File: breakout/breakout.kicad_sch (KiCad schematic)
At the start: 6 parts, among them J1 Conn_01x02, J2 Conn_01x04, J5 Conn_01x03

Commit message: Add 0805 decoupling capacitor pads to the breakout board.
Parts:
- added C1, C2: C, Capacitor_SMD:C_0805_2012Metric_Pad1.18x1.45mm_HandSolder, symbol Device:C
- J3, J4: value (none) -> Conn_01x05; footprint (none) -> Connector_PinHeader_2.54mm:PinHeader_1x05_P2.54mm_Vertical
- U1: value (none) -> 74HC4051; footprint (none) -> Package_SO:SO-16_5.3x10.2mm_P1.27mm
Connections:
- net GND: now also C1.2, C2.1
- net VCC: now also C2.2
- net VEE: now also C1.1
Other:
- moved on the sheet: J5
