File: pcb_6_muxes/multiplex.kicad_sch (KiCad schematic)
At the start: 4 parts, among them U1 74HC4051

Commit message: Re-layout with VEE=GND on 121mmx121mm single sided board.
Parts:
- added JOut1: Conn_01x01, Connector_PinHeader_2.54mm:PinHeader_1x01_P2.54mm_Vertical, symbol Connector_Generic:Conn_01x01
Connections:
- net OUT: no longer names the net of U1.3 (A)
- net OUT: now also JOut1.1 (Pin_1)
Changed lines of the file:
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@@
+    (stroke (width 0) (type default))
+  )
+  (wire (pts (xy 76.2 54.61) (xy 82.55 54.61))
     (stroke (width 0) (type default))
   )
@@
     (effects (font (size 1.27 1.27)) (justify right))
   )
-  (hierarchical_label "OUT" (shape output) (at 82.55 54.61 180) (fields_autoplaced)
-    (effects (font (size 1.27 1.27)) (justify right))
-  )
   (symbol (lib_id "Connector_Generic:Conn_01x03") (at 71.12 62.23 0) (mirror y) (unit 1)
     (in_bom yes) (on_board yes) (dnp no) (fields_autoplaced)
@@
           (reference "JSel1") (unit 1)
         )
-        (path "/011c74c2-4650-451f-bc3a-043fb00e6a79/78e9111b-39d6-4ab2-a0d0-9aa130c50d92"
+        (path "/011c74c2-4650-451f-bc3a-043fb00e6a79/bcdb0e81-b52f-4b9d-813e-9b54da9a2d97"
           (reference "JSel2") (unit 1)
         )
-        (path "/011c74c2-4650-451f-bc3a-043fb00e6a79/7adcadb4-5284-4cbe-8db6-9aa2f3595a86"
+        (path "/011c74c2-4650-451f-bc3a-043fb00e6a79/c13e9262-3ef2-4667-9ef1-27e6c11a7cc8"
           (reference "JSel3") (unit 1)
         )
-        (path "/011c74c2-4650-451f-bc3a-043fb00e6a79/e5bf1238-0ac0-4c51-a0a5-15b523661f91"
+        (path "/011c74c2-4650-451f-bc3a-043fb00e6a79/23a15acc-e1f8-4769-b83f-40cb177f8934"
           (reference "JSel4") (unit 1)
         )
-        (path "/011c74c2-4650-451f-bc3a-043fb00e6a79/40cbac75-c656-488a-b938-397f597f41f1"
+        (path "/011c74c2-4650-451f-bc3a-043fb00e6a79/a0bbbfe0-e56f-4670-85ad-77d23031e1c1"
           (reference "JSel5") (unit 1)
         )
-        (path "/011c74c2-4650-451f-bc3a-043fb00e6a79/87bc8edf-bd5c-406e-a98a-d85a01a66a70"
+        (path "/011c74c2-4650-451f-bc3a-043fb00e6a79/d37dde3d-e8b9-46fa-845e-b8126108a9ab"
           (reference "JSel6") (unit 1)
         )
@@
           (reference "JIn1") (unit 1)
         )
-        (path "/011c74c2-4650-451f-bc3a-043fb00e6a79/78e9111b-39d6-4ab2-a0d0-9aa130c50d92"
+        (path "/011c74c2-4650-451f-bc3a-043fb00e6a79/bcdb0e81-b52f-4b9d-813e-9b54da9a2d97"
           (reference "JIn3") (unit 1)
         )
-        (path "/011c74c2-4650-451f-bc3a-043fb00e6a79/7adcadb4-5284-4cbe-8db6-9aa2f3595a86"
+        (path "/011c74c2-4650-451f-bc3a-043fb00e6a79/c13e9262-3ef2-4667-9ef1-27e6c11a7cc8"
           (reference "JIn5") (unit 1)
         )
-        (path "/011c74c2-4650-451f-bc3a-043fb00e6a79/e5bf1238-0ac0-4c51-a0a5-15b523661f91"
+        (path "/011c74c2-4650-451f-bc3a-043fb00e6a79/23a15acc-e1f8-4769-b83f-40cb177f8934"
           (reference "JIn7") (unit 1)
         )
-        (path "/011c74c2-4650-451f-bc3a-043fb00e6a79/40cbac75-c656-488a-b938-397f597f41f1"
+        (path "/011c74c2-4650-451f-bc3a-043fb00e6a79/a0bbbfe0-e56f-4670-85ad-77d23031e1c1"
           (reference "JIn9") (unit 1)
         )
-        (path "/011c74c2-4650-451f-bc3a-043fb00e6a79/87bc8edf-bd5c-406e-a98a-d85a01a66a70"
+        (path "/011c74c2-4650-451f-bc3a-043fb00e6a79/d37dde3d-e8b9-46fa-845e-b8126108a9ab"
           (reference "JIn11") (unit 1)
         )
@@
     )
   )
+  (symbol (lib_id "Connector_Generic:Conn_01x01") (at 71.12 54.61 180) (unit 1)
+    (in_bom yes) (on_board yes) (dnp no) (fields_autoplaced)
+    (property "Reference" "JOut1" (at 71.12 48.26 0)
+      (effects (font (size 1.27 1.27)))
+    )
+    (property "Value" "Conn_01x01" (at 71.12 50.8 0)
+      (effects (font (size 1.27 1.27)))
+    )
+    (property "Footprint" "Connector_PinHeader_2.54mm:PinHeader_1x01_P2.54mm_Vertical" (at 71.12 54.61 0)
+      (effects (font (size 1.27 1.27)) hide)
+    )
+    (property "Datasheet" "~" (at 71.12 54.61 0)
+      (effects (font (size 1.27 1.27)) hide)
+    )
+    (pin "1")
+    (instances
+      (project "pcb_6_muxes"
+        (path "/011c74c2-4650-451f-bc3a-043fb00e6a79/1ee7e437-0e0d-4fe4-9554-b96bca794a00"
+          (reference "JOut1") (unit 1)
+        )
+        (path "/011c74c2-4650-451f-bc3a-043fb00e6a79/bcdb0e81-b52f-4b9d-813e-9b54da9a2d97"
+          (reference "JOut2") (unit 1)
+        )
+        (path "/011c74c2-4650-451f-bc3a-043fb00e6a79/c13e9262-3ef2-4667-9ef1-27e6c11a7cc8"
+          (reference "JOut3") (unit 1)
+        )
+        (path "/011c74c2-4650-451f-bc3a-043fb00e6a79/23a15acc-e1f8-4769-b83f-40cb177f8934"
+          (reference "JOut4") (unit 1)
+        )
+        (path "/011c74c2-4650-451f-bc3a-043fb00e6a79/a0bbbfe0-e56f-4670-85ad-77d23031e1c1"
+          (reference "JOut5") (unit 1)
+        )
+        (path "/011c74c2-4650-451f-bc3a-043fb00e6a79/d37dde3d-e8b9-46fa-845e-b8126108a9ab"
+          (reference "JOut6") (unit 1)
+        )
+      )
+    )
+  )
   (symbol (lib_id "Connector_Generic:Conn_01x04") (at 109.22 67.31 0) (unit 1)
     (in_bom yes) (on_board yes) (dnp no) (fields_autoplaced)
@@
           (reference "JIn2") (unit 1)
         )
-        (path "/011c74c2-4650-451f-bc3a-043fb00e6a79/78e9111b-39d6-4ab2-a0d0-9aa130c50d92"
+        (path "/011c74c2-4650-451f-bc3a-043fb00e6a79/bcdb0e81-b52f-4b9d-813e-9b54da9a2d97"
           (reference "JIn4") (unit 1)
         )
-        (path "/011c74c2-4650-451f-bc3a-043fb00e6a79/7adcadb4-5284-4cbe-8db6-9aa2f3595a86"
+        (path "/011c74c2-4650-451f-bc3a-043fb00e6a79/c13e9262-3ef2-4667-9ef1-27e6c11a7cc8"
           (reference "JIn6") (unit 1)
         )
-        (path "/011c74c2-4650-451f-bc3a-043fb00e6a79/e5bf1238-0ac0-4c51-a0a5-15b523661f91"
+        (path "/011c74c2-4650-451f-bc3a-043fb00e6a79/23a15acc-e1f8-4769-b83f-40cb177f8934"
           (reference "JIn8") (unit 1)
         )
-        (path "/011c74c2-4650-451f-bc3a-043fb00e6a79/40cbac75-c656-488a-b938-397f597f41f1"
+        (path "/011c74c2-4650-451f-bc3a-043fb00e6a79/a0bbbfe0-e56f-4670-85ad-77d23031e1c1"
           (reference "JIn10") (unit 1)
         )
-        (path "/011c74c2-4650-451f-bc3a-043fb00e6a79/87bc8edf-bd5c-406e-a98a-d85a01a66a70"
+        (path "/011c74c2-4650-451f-bc3a-043fb00e6a79/d37dde3d-e8b9-46fa-845e-b8126108a9ab"
           (reference "JIn12") (unit 1)
         )
@@
           (reference "U1") (unit 1)
         )
-        (path "/011c74c2-4650-451f-bc3a-043fb00e6a79/78e9111b-39d6-4ab2-a0d0-9aa130c50d92"
+        (path "/011c74c2-4650-451f-bc3a-043fb00e6a79/bcdb0e81-b52f-4b9d-813e-9b54da9a2d97"
           (reference "U2") (unit 1)
         )
-        (path "/011c74c2-4650-451f-bc3a-043fb00e6a79/7adcadb4-5284-4cbe-8db6-9aa2f3595a86"
+        (path "/011c74c2-4650-451f-bc3a-043fb00e6a79/c13e9262-3ef2-4667-9ef1-27e6c11a7cc8"
           (reference "U3") (unit 1)
         )
-        (path "/011c74c2-4650-451f-bc3a-043fb00e6a79/e5bf1238-0ac0-4c51-a0a5-15b523661f91"
+        (path "/011c74c2-4650-451f-bc3a-043fb00e6a79/23a15acc-e1f8-4769-b83f-40cb177f8934"
           (reference "U4") (unit 1)
         )
-        (path "/011c74c2-4650-451f-bc3a-043fb00e6a79/40cbac75-c656-488a-b938-397f597f41f1"
+        (path "/011c74c2-4650-451f-bc3a-043fb00e6a79/a0bbbfe0-e56f-4670-85ad-77d23031e1c1"
           (reference "U5") (unit 1)
         )
-        (path "/011c74c2-4650-451f-bc3a-043fb00e6a79/87bc8edf-bd5c-406e-a98a-d85a01a66a70"
+        (path "/011c74c2-4650-451f-bc3a-043fb00e6a79/d37dde3d-e8b9-46fa-845e-b8126108a9ab"
           (reference "U6") (unit 1)
         )
