File: pcb_6_muxes/pcb_6_muxes.kicad_sch (KiCad schematic)
At the start: 4 parts

Commit message: Re-layout with VEE=GND on 121mmx121mm single sided board.
Parts:
- removed C2: C, Capacitor_THT:C_Radial_D6.3mm_H5.0mm_P2.50mm, symbol Device:C
- removed JOut1: Conn_01x07, Connector_PinSocket_2.54mm:PinSocket_1x07_P2.54mm_Vertical, symbol Connector_Generic:Conn_01x07
- JPow1: value Conn_01x03 -> Conn_01x02; footprint Connector_PinHeader_2.54mm:PinHeader_1x03_P2.54mm_Vertical -> Connector_PinHeader_2.54mm:PinHeader_1x02_P2.54mm_Vertical; symbol Connector_Generic:Conn_01x03 -> Connector_Generic:Conn_01x02
Connections:
- removed net VEE: JPow1.3 (Pin_3)
Changed lines of the file:
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@@
   (junction (at 82.55 33.02) (diameter 0) (color 0 0 0 0)
-  )
-  (junction (at 82.55 43.18) (diameter 0) (color 0 0 0 0)
   )
   (wire (pts (xy 88.9 30.48) (xy 88.9 22.86))
@@
     (stroke (width 0) (type default))
   )
-  (wire (pts (xy 88.9 35.56) (xy 88.9 43.18))
-    (stroke (width 0) (type default))
-  )
   (wire (pts (xy 82.55 22.86) (xy 82.55 24.13))
     (stroke (width 0) (type default))
@@
     (stroke (width 0) (type default))
   )
-  (wire (pts (xy 88.9 43.18) (xy 82.55 43.18))
-    (stroke (width 0) (type default))
-  )
   (wire (pts (xy 81.28 33.02) (xy 82.55 33.02))
     (stroke (width 0) (type default))
@@
     (stroke (width 0) (type default))
   )
-  (wire (pts (xy 90.17 35.56) (xy 88.9 35.56))
-    (stroke (width 0) (type default))
-  )
   (wire (pts (xy 90.17 33.02) (xy 82.55 33.02))
-    (stroke (width 0) (type default))
-  )
-  (wire (pts (xy 82.55 41.91) (xy 82.55 43.18))
     (stroke (width 0) (type default))
   )
@@
     (effects (font (size 1.27 1.27)) (justify right bottom))
   )
-  (label "A1" (at 76.2 68.58 180) (fields_autoplaced)
-    (effects (font (size 1.27 1.27)) (justify right bottom))
-  )
-  (label "A5" (at 27.94 165.1 0) (fields_autoplaced)
-    (effects (font (size 1.27 1.27)) (justify left bottom))
-  )
-  (label "A0" (at 27.94 31.75 0) (fields_autoplaced)
-    (effects (font (size 1.27 1.27)) (justify left bottom))
-  )
-  (label "A2" (at 76.2 71.12 180) (fields_autoplaced)
-    (effects (font (size 1.27 1.27)) (justify right bottom))
-  )
-  (label "A5" (at 76.2 78.74 180) (fields_autoplaced)
-    (effects (font (size 1.27 1.27)) (justify right bottom))
-  )
-  (label "A2" (at 27.94 85.09 0) (fields_autoplaced)
-    (effects (font (size 1.27 1.27)) (justify left bottom))
-  )
-  (label "A1" (at 27.94 58.42 0) (fields_autoplaced)
-    (effects (font (size 1.27 1.27)) (justify left bottom))
-  )
-  (label "A3" (at 76.2 73.66 180) (fields_autoplaced)
-    (effects (font (size 1.27 1.27)) (justify right bottom))
-  )
-  (label "A0" (at 76.2 66.04 180) (fields_autoplaced)
-    (effects (font (size 1.27 1.27)) (justify right bottom))
-  )
-  (label "A4" (at 27.94 138.43 0) (fields_autoplaced)
-    (effects (font (size 1.27 1.27)) (justify left bottom))
-  )
-  (label "A4" (at 76.2 76.2 180) (fields_autoplaced)
-    (effects (font (size 1.27 1.27)) (justify right bottom))
-  )
-  (label "A3" (at 27.94 111.76 0) (fields_autoplaced)
-    (effects (font (size 1.27 1.27)) (justify left bottom))
-  )
   (symbol (lib_id "power:VCC") (at 27.94 114.3 270) (unit 1)
     (in_bom yes) (on_board yes) (dnp no)
@@
     )
   )
-  (symbol (lib_id "Connector_Generic:Conn_01x03") (at 95.25 33.02 0) (unit 1)
-    (in_bom yes) (on_board yes) (dnp no) (fields_autoplaced)
-    (property "Reference" "JPow1" (at 97.79 31.75 0)
-      (effects (font (size 1.27 1.27)) (justify left))
-    )
-    (property "Value" "Conn_01x03" (at 97.79 34.29 0)
-      (effects (font (size 1.27 1.27)) (justify left))
-    )
-    (property "Footprint" "Connector_PinHeader_2.54mm:PinHeader_1x03_P2.54mm_Vertical" (at 95.25 33.02 0)
-      (effects (font (size 1.27 1.27)) hide)
-    )
-    (property "Datasheet" "~" (at 95.25 33.02 0)
+  (symbol (lib_id "Connector_Generic:Conn_01x02") (at 95.25 30.48 0) (unit 1)
+    (in_bom yes) (on_board yes) (dnp no) (fields_autoplaced)
+    (property "Reference" "JPow1" (at 97.79 29.21 0)
+      (effects (font (size 1.27 1.27)) (justify left))
+    )
+    (property "Value" "Conn_01x02" (at 97.79 31.75 0)
+      (effects (font (size 1.27 1.27)) (justify left))
+    )
+    (property "Footprint" "Connector_PinHeader_2.54mm:PinHeader_1x02_P2.54mm_Vertical" (at 95.25 30.48 0)
+      (effects (font (size 1.27 1.27)) hide)
+    )
+    (property "Datasheet" "~" (at 95.25 30.48 0)
       (effects (font (size 1.27 1.27)) hide)
     )
     (pin "1")
     (pin "2")
-    (pin "3")
     (instances
       (project "pcb_6_muxes"
@@
     )
   )
-  (symbol (lib_id "Connector_Generic:Conn_01x07") (at 81.28 73.66 0) (unit 1)
-    (in_bom yes) (on_board yes) (dnp no) (fields_autoplaced)
-    (property "Reference" "JOut1" (at 83.82 72.39 0)
-      (effects (font (size 1.27 1.27)) (justify left))
-    )
-    (property "Value" "Conn_01x07" (at 83.82 74.93 0)
-      (effects (font (size 1.27 1.27)) (justify left))
-    )
-    (property "Footprint" "Connector_PinSocket_2.54mm:PinSocket_1x07_P2.54mm_Vertical" (at 81.28 73.66 0)
-      (effects (font (size 1.27 1.27)) hide)
-    )
-    (property "Datasheet" "~" (at 81.28 73.66 0)
-      (effects (font (size 1.27 1.27)) hide)
-    )
-    (pin "1")
-    (pin "2")
-    (pin "3")
-    (pin "4")
-    (pin "5")
-    (pin "6")
-    (pin "7")
-    (instances
-      (project "pcb_6_muxes"
-        (path "/011c74c2-4650-451f-bc3a-043fb00e6a79"
-          (reference "JOut1") (unit 1)
-        )
-      )
-    )
-  )
   (symbol (lib_id "power:GND") (at 27.94 152.4 90) (unit 1)
     (in_bom yes) (on_board yes) (dnp no) (fields_autoplaced)
@@
     )
   )
-  (symbol (lib_id "Device:C") (at 82.55 38.1 0) (unit 1)
-    (in_bom yes) (on_board yes) (dnp no) (fields_autoplaced)
-    (property "Reference" "C2" (at 86.36 36.83 0)
-      (effects (font (size 1.27 1.27)) (justify left))
-    )
-    (property "Value" "C" (at 86.36 39.37 0)
-      (effects (font (size 1.27 1.27)) (justify left))
-    )
-    (property "Footprint" "Capacitor_THT:C_Radial_D6.3mm_H5.0mm_P2.50mm" (at 83.5152 41.91 0)
-      (effects (font (size 1.27 1.27)) hide)
-    )
-    (property "Datasheet" "~" (at 82.55 38.1 0)
-      (effects (font (size 1.27 1.27)) hide)
-    )
-    (pin "1")
-    (pin "2")
-    (instances
-      (project "pcb_6_muxes"
-        (path "/011c74c2-4650-451f-bc3a-043fb00e6a79"
-          (reference "C2") (unit 1)
-        )
-      )
-    )
-  )
   (symbol (lib_id "power:GND") (at 27.94 125.73 90) (unit 1)
     (in_bom yes) (on_board yes) (dnp no) (fields_autoplaced)
@@
     )
   )
-  (symbol (lib_id "power:VEE") (at 82.55 43.18 180) (unit 1)
+  (symbol (lib_id "power:VEE") (at 82.55 34.29 180) (unit 1)
     (in_bom yes) (on_board yes) (dnp no)
-    (property "Reference" "#PWR021" (at 82.55 39.37 0)
-      (effects (font (size 1.27 1.27)) hide)
-    )
-    (property "Value" "VEE" (at 82.5499 46.99 90)
-      (effects (font (size 1.27 1.27)) (justify left))
-    )
-    (property "Footprint" "" (at 82.55 43.18 0)
-      (effects (font (size 1.27 1.27)) hide)
-    )
-    (property "Datasheet" "" (at 82.55 43.18 0)
+    (property "Reference" "#PWR021" (at 82.55 30.48 0)
+      (effects (font (size 1.27 1.27)) hide)
+    )
+    (property "Value" "VEE" (at 82.5499 38.1 90)
+      (effects (font (size 1.27 1.27)) (justify left))
+    )
+    (property "Footprint" "" (at 82.55 34.29 0)
+      (effects (font (size 1.27 1.27)) hide)
+    )
+    (property "Datasheet" "" (at 82.55 34.29 0)
       (effects (font (size 1.27 1.27)) hide)
     )
@@
         (path "/011c74c2-4650-451f-bc3a-043fb00e6a79"
           (reference "#PWR010") (unit 1)
-        )
-      )
-    )
-  )
-  (symbol (lib_id "power:GND") (at 76.2 81.28 270) (unit 1)
-    (in_bom yes) (on_board yes) (dnp no) (fields_autoplaced)
-    (property "Reference" "#PWR022" (at 69.85 81.28 0)
-      (effects (font (size 1.27 1.27)) hide)
-    )
-    (property "Value" "GND" (at 72.39 81.28 90)
-      (effects (font (size 1.27 1.27)) (justify right))
-    )
-    (property "Footprint" "" (at 76.2 81.28 0)
-      (effects (font (size 1.27 1.27)) hide)
-    )
-    (property "Datasheet" "" (at 76.2 81.28 0)
-      (effects (font (size 1.27 1.27)) hide)
-    )
-    (pin "1")
-    (instances
-      (project "pcb_6_muxes"
-        (path "/011c74c2-4650-451f-bc3a-043fb00e6a79"
-          (reference "#PWR022") (unit 1)
         )
       )
@@
     )
   )
+  (sheet (at 15.24 96.52) (size 12.7 20.32) (fields_autoplaced)
+    (stroke (width 0.1524) (type solid))
+    (fill (color 0 0 0 0.0000))
+    (property "Sheetname" "Multiplex4" (at 15.24 95.8084 0)
+      (effects (font (size 1.27 1.27)) (justify left bottom))
+    )
+    (property "Sheetfile" "multiplex.kicad_sch" (at 15.24 117.4246 0)
+      (effects (font (size 1.27 1.27)) (justify left top))
+    )
+    (pin "VCC" input (at 27.94 114.3 0)
+      (effects (font (size 1.27 1.27)) (justify right))
+    )
+    (pin "OUT" output (at 27.94 111.76 0)
+      (effects (font (size 1.27 1.27)) (justify right))
+    )
+    (pin "VEE" input (at 27.94 101.6 0)
+      (effects (font (size 1.27 1.27)) (justify right))
+    )
+    (pin "GND" input (at 27.94 99.06 0)
+      (effects (font (size 1.27 1.27)) (justify right))
+    )
+    (instances
+      (project "pcb_6_muxes"
+        (path "/011c74c2-4650-451f-bc3a-043fb00e6a79" (page "5"))
+      )
+    )
+  )
   (sheet (at 15.24 123.19) (size 12.7 20.32) (fields_autoplaced)
     (stroke (width 0.1524) (type solid))
@@
       )
     )
-  )
-  (sheet (at 15.24 96.52) (size 12.7 20.32) (fields_autoplaced)
-    (stroke (width 0.1524) (type solid))
-    (fill (color 0 0 0 0.0000))
-    (property "Sheetname" "Multiplex4" (at 15.24 95.8084 0)
-      (effects (font (size 1.27 1.27)) (justify left bottom))
-    )
-    (property "Sheetfile" "multiplex.kicad_sch" (at 15.24 117.4246 0)
-      (effects (font (size 1.27 1.27)) (justify left top))
-    )
-    (pin "VCC" input (at 27.94 114.3 0)
-      (effects (font (size 1.27 1.27)) (justify right))
-    )
-    (pin "OUT" output (at 27.94 111.76 0)
-      (effects (font (size 1.27 1.27)) (justify right))
-    )
-    (pin "VEE" input (at 27.94 101.6 0)
-      (effects (font (size 1.27 1.27)) (justify right))
-    )
-    (pin "GND" input (at 27.94 99.06 0)
-      (effects (font (size 1.27 1.27)) (justify right))
-    )
-    (instances
-      (project "pcb_6_muxes"
-        (path "/011c74c2-4650-451f-bc3a-043fb00e6a79" (page "5"))
-      )
-    )
